Commit message: fix sentry

File: rm_gimbal_description/urdf/rm_gimbal.urdf.xacro (robot description, xacro)
@@ -2,10 +2,10 @@
 <robot name="rm_gimbal"
   xmlns:xacro="http://ros.org/wiki/xacro">
-  <xacro:arg name="xyz" default="0.10 0 0.03" />
+  <xacro:arg name="xyz" default="0.10 0 -0.01" />
   <xacro:arg name="rpy" default="0 0 0" />
-  <link name="odom" />
+  <link name="gimbal_imu" />
   <link name="gimbal_link" />
   <joint name="gimbal_joint" type="floating">
-    <parent link="odom" />
+    <parent link="gimbal_imu" />
     <child link="gimbal_link" />
   </joint>

Commit message: change URDF

File: rm_gimbal_description/urdf/rm_gimbal.urdf.xacro (robot description, xacro)
@@ -5,20 +5,35 @@
   <xacro:arg name="rpy" default="0 0 0" />
   <link name="odom" />
-  <link name="gimbal_link" />
-  <joint name="gimbal_joint" type="floating">
+  <link name="yaw_link" />
+  <joint name="yaw_joint" type="continuous">
     <parent link="odom" />
-    <child link="gimbal_link" />
+    <child link="yaw_link" />
+    <axis xyz="0 0 1" />
+  </joint>
+  <link name="pitch_link" />
+  <joint name="pitch_joint" type="continuous">
+    <parent link="yaw_link" />
+    <child link="pitch_link" />
+    <origin xyz="-0.06 0 0.15" rpy="0 0 0" />
+    <axis xyz="0 1 0" />
   </joint>
   <link name="camera_link" />
   <joint name="camera_joint" type="fixed">
     <origin xyz="$(arg xyz)" rpy="$(arg rpy)" />
-    <parent link="gimbal_link" />
+    <parent link="pitch_link" />
     <child link="camera_link" />
-    <axis xyz="0 0 0" />
+    <!-- <axis xyz="0 0 0" /> -->
+  </joint>
+  <link name="virtual_pitch"/>
+  <joint name="virtual_pitch_joint" type="fixed">
+    <origin xyz="0 0 0" rpy="0 0.2413 0" />
+    <parent link="camera_link" />
+    <child link="virtual_pitch" />
   </joint>
   <link name="camera_optical_frame" />
   <joint name="camera_optical_joint" type="fixed">
+  <!-- hero -->
     <origin xyz="0 0 0" rpy="${-pi/2} 0 ${-pi/2}" />
-    <parent link="camera_link" />
+    <parent link="virtual_pitch" />
     <child link="camera_optical_frame" />
   </joint>

Commit message: change URDF

File: rm_gimbal_description/urdf/rm_gimbal.urdf.xacro (robot description, xacro)
@@ -2,23 +2,38 @@
 <robot name="rm_gimbal"
   xmlns:xacro="http://ros.org/wiki/xacro">
-  <xacro:arg name="xyz" default="0.10 0.0 0.075" />
+  <xacro:arg name="xyz" default="0.10 0 0.03" />
   <xacro:arg name="rpy" default="0 0 0" />
   <link name="odom" />
-  <link name="gimbal_link" />
-  <joint name="gimbal_joint" type="floating">
+  <link name="yaw_link" />
+  <joint name="yaw_joint" type="continuous">
     <parent link="odom" />
-    <child link="gimbal_link" />
+    <child link="yaw_link" />
+    <axis xyz="0 0 1" />
+  </joint>
+  <link name="pitch_link" />
+  <joint name="pitch_joint" type="continuous">
+    <parent link="yaw_link" />
+    <child link="pitch_link" />
+    <origin xyz="0 0 0.15" rpy="0 0 0" />
+    <axis xyz="0 1 0" />
   </joint>
   <link name="camera_link" />
   <joint name="camera_joint" type="fixed">
     <origin xyz="$(arg xyz)" rpy="$(arg rpy)" />
-    <parent link="gimbal_link" />
+    <parent link="pitch_link" />
     <child link="camera_link" />
-    <axis xyz="0 0 0" />
+    <!-- <axis xyz="0 0 0" /> -->
+  </joint>
+  <link name="virtual_pitch"/>
+  <joint name="virtual_pitch_joint" type="fixed">
+    <origin xyz="0 0 0" rpy="0 0.2413 0" />
+    <parent link="camera_link" />
+    <child link="virtual_pitch" />
   </joint>
   <link name="camera_optical_frame" />
   <joint name="camera_optical_joint" type="fixed">
+  <!-- hero -->
     <origin xyz="0 0 0" rpy="${-pi/2} 0 ${-pi/2}" />
-    <parent link="camera_link" />
+    <parent link="virtual_pitch" />
     <child link="camera_optical_frame" />
   </joint>

Commit message: change URDF

File: rm_gimbal_description/urdf/rm_gimbal.urdf.xacro (robot description, xacro)
@@ -15,5 +15,5 @@
     <parent link="yaw_link" />
     <child link="pitch_link" />
-    <origin xyz="0 0 0.15" rpy="0 0 0" />
+    <origin xyz="0 0 0.20" rpy="0 0 0" />
     <axis xyz="0 1 0" />
   </joint>

Commit message: change URDF

File: rm_gimbal_description/urdf/rm_gimbal.urdf.xacro (robot description, xacro)
@@ -20,14 +20,7 @@
   <link name="camera_link" />
   <joint name="camera_joint" type="fixed">
-    <origin xyz="$(arg xyz)" rpy="$(arg rpy)" />
+    <origin xyz="0.12 0 0.08" rpy="$(arg rpy)" />
     <parent link="pitch_link" />
     <child link="camera_link" />
-    <!-- <axis xyz="0 0 0" /> -->
-  </joint>
-  <link name="virtual_pitch"/>
-  <joint name="virtual_pitch_joint" type="fixed">
-    <origin xyz="0 0 0" rpy="0 0.2413 0" />
-    <parent link="camera_link" />
-    <child link="virtual_pitch" />
   </joint>
   <link name="camera_optical_frame" />
@@ -35,5 +28,5 @@
   <!-- hero -->
     <origin xyz="0 0 0" rpy="${-pi/2} 0 ${-pi/2}" />
-    <parent link="virtual_pitch" />
+    <parent link="camera_link" />
     <child link="camera_optical_frame" />
   </joint>

Commit message: solve trajectory bug

File: rm_gimbal_description/urdf/rm_gimbal.urdf.xacro (robot description, xacro)
@@ -15,5 +15,7 @@
     <parent link="yaw_link" />
     <child link="pitch_link" />
-    <origin xyz="0 0 0.20" rpy="0 0 0" />
+    <!-- <origin xyz="0 0 0.20" rpy="0 0 0" /> -->
+    <!-- 实际决定这里的是serial driver -->
+    <origin xyz="0 0 0.0" rpy="0 0 0" />
     <axis xyz="0 1 0" />
   </joint>

Commit message: correct URDF

File: rm_gimbal_description/urdf/rm_gimbal.urdf.xacro (robot description, xacro)
@@ -5,13 +5,21 @@
   <xacro:arg name="rpy" default="0 0 0" />
   <link name="gimbal_imu" />
-  <link name="gimbal_link" />
-  <joint name="gimbal_joint" type="floating">
+  <link name="yaw_link" />
+  <joint name="yaw_joint" type="continuous">
     <parent link="gimbal_imu" />
-    <child link="gimbal_link" />
+    <child link="yaw_link" />
+    <axis xyz="0 0 1" />
+  </joint>
+  <link name="pitch_link" />
+  <joint name="pitch_joint" type="continuous">
+    <parent link="yaw_link" />
+    <child link="pitch_link" />
+    <origin xyz="-0.06 0 0.15" rpy="0 0 0" />
+    <axis xyz="0 1 0" />
   </joint>
   <link name="camera_link" />
   <joint name="camera_joint" type="fixed">
     <origin xyz="$(arg xyz)" rpy="$(arg rpy)" />
-    <parent link="gimbal_link" />
+    <parent link="pitch_link" />
     <child link="camera_link" />
     <axis xyz="0 0 0" />

Commit message: change tracker

File: rm_gimbal_description/urdf/rm_gimbal.urdf.xacro (robot description, xacro)
@@ -20,5 +20,5 @@
   <link name="camera_link" />
   <joint name="camera_joint" type="fixed">
-    <origin xyz="$(arg xyz)" rpy="$(arg rpy)" />
+    <origin xyz="0.08 0 0.11" rpy="$(arg rpy)" />
     <parent link="pitch_link" />
     <child link="camera_link" />
